Commit message: tweaked urdf with top-of-my-head inertias and masses, but with proper sizes and stl files

File: src/khan_description/urdf/decorations.urdf.xacro (robot description, xacro)
@@ -28,5 +28,5 @@
         <origin xyz="0 0 0" rpy="0 0 0" />
         <geometry>
-          <mesh filename="package://khan_description/meshes/top_chassis.dae" />
+          <mesh filename="package://khan_description/meshes/top_chassis.stl" />
         </geometry>
       </visual>
@@ -41,5 +41,5 @@
       <visual>
         <geometry>
-          <mesh filename="package://khan_description/meshes/user_rail.dae" />
+          <mesh filename="package://khan_description/meshes/user_rail.stl" />
         </geometry>
       </visual>
@@ -55,5 +55,5 @@
       <visual>
         <geometry>
-          <mesh filename="package://khan_description/meshes/bumper.dae" />
+          <mesh filename="package://khan_description/meshes/bumper.stl" />
         </geometry>
       </visual>
@@ -69,5 +69,5 @@
       <visual>
         <geometry>
-          <mesh filename="package://khan_description/meshes/bumper.dae" />
+          <mesh filename="package://khan_description/meshes/bumper.stl" />
         </geometry>
       </visual>
@@ -85,5 +85,5 @@
           <origin xyz="0 0 0" rpy="0 0 0" />
           <geometry>
-            <mesh filename="package://khan_description/meshes/top_plate.dae" />
+            <mesh filename="package://khan_description/meshes/top_plate.stl" />
           </geometry>
         </visual>
@@ -91,5 +91,5 @@
           <origin xyz="0 0 0" rpy="0 0 0"/>
           <geometry>
-            <mesh filename="package://khan_description/meshes/top_plate.dae" />
+            <mesh filename="package://khan_description/meshes/top_plate.stl" />
           </geometry>
         </collision>

File: src/khan_description/urdf/khan.urdf.xacro (robot description, xacro)
@@ -27,33 +27,28 @@
   <property name="M_PI" value="3.14159"/>
   <!-- Base Size -->
-  <property name="base_x_size" value="0.98740000" />
-  <property name="base_y_size" value="0.57090000" />
-  <property name="base_z_size" value="0.24750000" />
+  <property name="base_x_size" value="0.245" />
+  <property name="base_y_size" value="0.153" />
+  <property name="base_z_size" value="0.074" />
+  <property name="base_z_clearance" value="0.021" />
   <!-- Wheel Mounting Positions -->
-  <xacro:property name="wheelbase" value="0.5120" />
-  <xacro:property name="track" value="0.5708" />
-  <xacro:property name="wheel_vertical_offset" value="0.03282" />
+  <xacro:property name="wheelbase" value="0.185" />
+  <xacro:property name="track" value="0.189" />
+  <xacro:property name="wheel_vertical_offset" value="0.0" />
   <!-- Wheel Properties -->
-  <xacro:property name="wheel_length" value="0.1143" />
-  <xacro:property name="wheel_radius" value="0.17775" />
+  <xacro:property name="wheel_length" value="0.036" />
+  <xacro:property name="wheel_radius" value="0.03" />
   <xacro:macro name="khan_robot">
-    <!-- Base link is the center of the robot's bottom plate -->
+    <!-- Base link is the center of the robot's base on ground -->
     <link name="base_link">
       <visual>
         <origin xyz="0 0 0" rpy="0 0 0" />
         <geometry>
-          <mesh filename="package://khan_description/meshes/base_link.dae" />
+          <mesh filename="package://khan_description/cad/rover_base_with_tread.stl" scale="0.001 0.001 0.001"/>
         </geometry>
       </visual>
-      <collision>
-        <origin xyz="0 0 ${base_z_size/4}" rpy="0 0 0" />
+      <collision> <!--FIXME-->
+        <origin xyz="0 0 ${base_z_clearance/2+base_z_size/2}" rpy="0 0 0" />
         <geometry>
-          <box size="${base_x_size} ${base_y_size} ${base_z_size/2}"/>
-        </geometry>
-      </collision>
-      <collision>
-        <origin xyz="0 0 ${base_z_size*3/4}" rpy="0 0 0" />
-        <geometry>
-          <box size="${base_x_size*4/5} ${base_y_size} ${base_z_size/2}"/>
+          <box size="${base_x_size} ${base_y_size} ${base_z_size-base_z_clearance}"/>
         </geometry>
       </collision>
@@ -62,14 +57,14 @@
     <link name="base_footprint"/>
     <joint name="base_footprint_joint" type="fixed">
-      <origin xyz="0 0 ${wheel_vertical_offset - wheel_radius}" rpy="0 0 0" />
+      <origin xyz="0 0 0" rpy="0 0 0" />
       <parent link="base_link" />
       <child link="base_footprint" />
     </joint>
     <!-- Interial link stores the robot's inertial information -->
-    <link name="inertial_link">
+    <link name="inertial_link"> <!--FIXME currently made up -->
       <inertial>
-        <mass value="33.455" />
-        <origin xyz="-0.08748 -0.00085 0.09947" />
-        <inertia ixx="0.6022" ixy="-0.02364" ixz="-0.1197" iyy="1.7386" iyz="-0.001544" izz="2.0296" />
+        <mass value="0.8" />
+        <origin xyz="0.0 0.0 0.035" />
+        <inertia ixx="0.1" ixy="-0.001" ixz="-0.001" iyy="0.3" iyz="-0.0001" izz="0.3" />
       </inertial>
     </link>
@@ -81,16 +76,16 @@
     <!-- Khan wheel macros -->
     <xacro:khan_wheel wheel_prefix="front_left">
-      <origin xyz="${wheelbase/2} ${track/2} ${wheel_vertical_offset}" rpy="0 0 0" />
+      <origin xyz="${wheelbase/2} ${track/2} ${wheel_radius}" rpy="0 0 0" />
     </xacro:khan_wheel>
     <xacro:khan_wheel wheel_prefix="front_right">
-      <origin xyz="${wheelbase/2} ${-track/2} ${wheel_vertical_offset}" rpy="0 0 0" />
+      <origin xyz="${wheelbase/2} ${-track/2} ${wheel_radius}" rpy="0 0 0" />
     </xacro:khan_wheel>
     <xacro:khan_wheel wheel_prefix="rear_left">
-      <origin xyz="${-wheelbase/2} ${track/2} ${wheel_vertical_offset}" rpy="0 0 0" />
+      <origin xyz="${-wheelbase/2} ${track/2} ${wheel_radius}" rpy="0 0 0" />
     </xacro:khan_wheel>
     <xacro:khan_wheel wheel_prefix="rear_right">
-      <origin xyz="${-wheelbase/2} ${-track/2} ${wheel_vertical_offset}" rpy="0 0 0" />
+      <origin xyz="${-wheelbase/2} ${-track/2} ${wheel_radius}" rpy="0 0 0" />
     </xacro:khan_wheel>
-    <xacro:khan_decorate />
+<!--    <xacro:khan_decorate /> FIXME -->
   </xacro:macro>
 </robot>

File: src/khan_description/urdf/wheel.urdf.xacro (robot description, xacro)
@@ -24,13 +24,13 @@
 	<xacro:macro name="khan_wheel" params="wheel_prefix *joint_pose">
 		<link name="${wheel_prefix}_wheel_link">
-			<inertial>
-				<mass value="2.637" />
+			<inertial> <!-- FIXME -->
+				<mass value=".05" />
 				<origin xyz="0 0 0" />
-				<inertia  ixx="0.02467" ixy="0" ixz="0" iyy="0.02467" iyz="0" izz="0.04411" />
+				<inertia  ixx="0.002" ixy="0" ixz="0" iyy="0.002" iyz="0" izz="0.004" />
 			</inertial>
 			<visual>
 				<origin xyz="0 0 0" rpy="0 0 0" />
 				<geometry>
-					<mesh filename="package://khan_description/meshes/wheel.dae" />
+					<mesh filename="package://khan_description/cad/rover_wheel.stl" scale="0.001 0.001 0.001" />
 				</geometry>
 			</visual>
