Commit message: modified urdf to locate stls in /meshes

File: src/khan_description/urdf/khan.urdf.xacro (robot description, xacro)
@@ -44,5 +44,5 @@
         <origin xyz="0 0 0" rpy="0 0 0" />
         <geometry>
-          <mesh filename="package://khan_description/cad/rover_base_with_tread.stl" scale="0.001 0.001 0.001"/>
+          <mesh filename="package://khan_description/meshes/rover_base_with_tread.stl" scale="0.001 0.001 0.001"/>
         </geometry>
       </visual>

File: src/khan_description/urdf/wheel.urdf.xacro (robot description, xacro)
@@ -32,5 +32,5 @@
 				<origin xyz="0 0 0" rpy="0 0 0" />
 				<geometry>
-					<mesh filename="package://khan_description/cad/rover_wheel.stl" scale="0.001 0.001 0.001" />
+					<mesh filename="package://khan_description/meshes/rover_wheel.stl" scale="0.001 0.001 0.001" />
 				</geometry>
 			</visual>
